File: docs/test-platform/test-platform.kicad_sch (KiCad schematic)
At the start: 24 parts, among them J1 Raspberry_Pi_40pin, M1 ADS1115_0x48, M2 ADS1115_0x49, M3 DS3231_ZS042, M4 BMP180, M5 SSD1306_OLED, M6 BSS138_LLC, M7 ULN2003_28BYJ48, M8 LCD_HD44780, U1 MCP23017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

Commit message: Assign generated footprints and validate KiCad schematic-to-PCB transfer
Parts:
- A1: footprint (none) -> test-platform:A1
- J1: footprint (none) -> test-platform:J1
- M1: footprint (none) -> test-platform:M1
- M2: footprint (none) -> test-platform:M2
- M3: footprint (none) -> test-platform:M3
- M4: footprint (none) -> test-platform:M4
- M5: footprint (none) -> test-platform:M5
- M6: footprint (none) -> test-platform:M6
- M7: footprint (none) -> test-platform:M7
- M8: footprint (none) -> test-platform:M8
- R1: footprint (none) -> test-platform:R1
- R2: footprint (none) -> test-platform:R2
- R3: footprint (none) -> test-platform:R3
- R4: footprint (none) -> test-platform:R4
- R5: footprint (none) -> test-platform:R5
- R6: footprint (none) -> test-platform:R6
- R7: footprint (none) -> test-platform:R7
- RV1: footprint (none) -> test-platform:RV1
- SV1: footprint (none) -> test-platform:SV1
- U1: footprint (none) -> test-platform:U1
- U2: footprint (none) -> test-platform:U2
- U3: footprint (none) -> test-platform:U3
- U4: footprint (none) -> test-platform:U4
- U5: footprint (none) -> test-platform:U5
Changed lines of the file:
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@@
     (property "Value" "Raspberry_Pi_40pin" (at 70.0000 80.8800 0)
       (effects (font (size 1.27 1.27))))
-    (property "Footprint" "" (at 70.0000 51.6700 0)
+    (property "Footprint" "test-platform:J1" (at 70.0000 51.6700 0)
       (effects (font (size 1.27 1.27)) hide))
     (property "Datasheet" "" (at 70.0000 51.6700 0)
@@
     (property "Value" "MCP23017" (at 180.0000 63.1000 0)
       (effects (font (size 1.27 1.27))))
-    (property "Footprint" "" (at 180.0000 42.7800 0)
+    (property "Footprint" "test-platform:U1" (at 180.0000 42.7800 0)
       (effects (font (size 1.27 1.27)) hide))
     (property "Datasheet" "" (at 180.0000 42.7800 0)
@@
     (property "Value" "74HC595" (at 180.0000 103.9600 0)
       (effects (font (size 1.27 1.27))))
-    (property "Footprint" "" (at 180.0000 89.9900 0)
+    (property "Footprint" "test-platform:U2" (at 180.0000 89.9900 0)
       (effects (font (size 1.27 1.27)) hide))
     (property "Datasheet" "" (at 180.0000 89.9900 0)
@@
     (property "Value" "MCP3008" (at 180.0000 144.8200 0)
       (effects (font (size 1.27 1.27))))
-    (property "Footprint" "" (at 180.0000 130.8500 0)
+    (property "Footprint" "test-platform:U3" (at 180.0000 130.8500 0)
       (effects (font (size 1.27 1.27)) hide))
     (property "Datasheet" "" (at 180.0000 130.8500 0)
@@
     (property "Value" "MCP4922" (at 180.0000 180.6000 0)
       (effects (font (size 1.27 1.27))))
-    (property "Footprint" "" (at 180.0000 169.1700 0)
+    (property "Footprint" "test-platform:U4" (at 180.0000 169.1700 0)
       (effects (font (size 1.27 1.27)) hide))
     (property "Datasheet" "" (at 180.0000 169.1700 0)
@@
     (property "Value" "MCP42010" (at 180.0000 218.9200 0)
       (effects (font (size 1.27 1.27))))
-    (property "Footprint" "" (at 180.0000 206.2200 0)
+    (property "Footprint" "test-platform:U5" (at 180.0000 206.2200 0)
       (effects (font (size 1.27 1.27)) hide))
     (property "Datasheet" "" (at 180.0000 206.2200 0)
@@
     (property "Value" "ADS1115_0x48" (at 180.0000 252.1600 0)
       (effects (font (size 1.27 1.27))))
-    (property "Footprint" "" (at 180.0000 242.0000 0)
+    (property "Footprint" "test-platform:M1" (at 180.0000 242.0000 0)
       (effects (font (size 1.27 1.27)) hide))
     (property "Datasheet" "" (at 180.0000 242.0000 0)
@@
     (property "Value" "ADS1115_0x49" (at 180.0000 285.4000 0)
       (effects (font (size 1.27 1.27))))
-    (property "Footprint" "" (at 180.0000 275.2400 0)
+    (property "Footprint" "test-platform:M2" (at 180.0000 275.2400 0)
       (effects (font (size 1.27 1.27)) hide))
     (property "Datasheet" "" (at 180.0000 275.2400 0)
@@
     (property "Value" "DS3231_ZS042" (at 180.0000 313.5600 0)
       (effects (font (size 1.27 1.27))))
-    (property "Footprint" "" (at 180.0000 305.9400 0)
+    (property "Footprint" "test-platform:M3" (at 180.0000 305.9400 0)
       (effects (font (size 1.27 1.27)) hide))
     (property "Datasheet" "" (at 180.0000 305.9400 0)
@@
     (property "Value" "BMP180" (at 180.0000 339.1800 0)
       (effects (font (size 1.27 1.27))))
-    (property "Footprint" "" (at 180.0000 332.8300 0)
+    (property "Footprint" "test-platform:M4" (at 180.0000 332.8300 0)
       (effects (font (size 1.27 1.27)) hide))
     (property "Datasheet" "" (at 180.0000 332.8300 0)
@@
     (property "Value" "SSD1306_OLED" (at 280.0000 35.1600 0)
       (effects (font (size 1.27 1.27))))
-    (property "Footprint" "" (at 280.0000 28.8100 0)
+    (property "Footprint" "test-platform:M5" (at 280.0000 28.8100 0)
       (effects (font (size 1.27 1.27)) hide))
     (property "Datasheet" "" (at 280.0000 28.8100 0)
@@
     (property "Value" "BSS138_LLC" (at 280.0000 65.8600 0)
       (effects (font (size 1.27 1.27))))
-    (property "Footprint" "" (at 280.0000 56.9700 0)
+    (property "Footprint" "test-platform:M6" (at 280.0000 56.9700 0)
       (effects (font (size 1.27 1.27)) hide))
     (property "Datasheet" "" (at 280.0000 56.9700 0)
@@
     (property "Value" "ULN2003_28BYJ48" (at 280.0000 94.0200 0)
       (effects (font (size 1.27 1.27))))
-    (property "Footprint" "" (at 280.0000 86.4000 0)
+    (property "Footprint" "test-platform:M7" (at 280.0000 86.4000 0)
       (effects (font (size 1.27 1.27)) hide))
     (property "Datasheet" "" (at 280.0000 86.4000 0)
@@
     (property "Value" "LCD_HD44780" (at 280.0000 129.8000 0)
       (effects (font (size 1.27 1.27))))
-    (property "Footprint" "" (at 280.0000 118.3700 0)
+    (property "Footprint" "test-platform:M8" (at 280.0000 118.3700 0)
       (effects (font (size 1.27 1.27)) hide))
     (property "Datasheet" "" (at 280.0000 118.3700 0)
@@
     (property "Value" "Arduino_MetroMini" (at 280.0000 155.4200 0)
       (effects (font (size 1.27 1.27))))
-    (property "Footprint" "" (at 280.0000 149.0700 0)
+    (property "Footprint" "test-platform:A1" (at 280.0000 149.0700 0)
       (effects (font (size 1.27 1.27)) hide))
     (property "Datasheet" "" (at 280.0000 149.0700 0)
@@
     (property "Value" "Servo" (at 280.0000 181.0400 0)
       (effects (font (size 1.27 1.27))))
-    (property "Footprint" "" (at 280.0000 174.6900 0)
+    (property "Footprint" "test-platform:SV1" (at 280.0000 174.6900 0)
       (effects (font (size 1.27 1.27)) hide))
     (property "Datasheet" "" (at 280.0000 174.6900 0)
@@
     (property "Value" "10k_pot" (at 280.0000 206.6600 0)
       (effects (font (size 1.27 1.27))))
-    (property "Footprint" "" (at 280.0000 200.3100 0)
+    (property "Footprint" "test-platform:RV1" (at 280.0000 200.3100 0)
       (effects (font (size 1.27 1.27)) hide))
     (property "Datasheet" "" (at 280.0000 200.3100 0)
@@
     (property "Value" "LDR" (at 280.0000 229.7400 0)
       (effects (font (size 1.27 1.27))))
-    (property "Footprint" "" (at 280.0000 224.6600 0)
+    (property "Footprint" "test-platform:R1" (at 280.0000 224.6600 0)
       (effects (font (size 1.27 1.27)) hide))
     (property "Datasheet" "" (at 280.0000 224.6600 0)
@@
     (property "Value" "LDR" (at 280.0000 252.8200 0)
       (effects (font (size 1.27 1.27))))
-    (property "Footprint" "" (at 280.0000 247.7400 0)
+    (property "Footprint" "test-platform:R2" (at 280.0000 247.7400 0)
       (effects (font (size 1.27 1.27)) hide))
     (property "Datasheet" "" (at 280.0000 247.7400 0)
@@
     (property "Value" "LDR" (at 280.0000 275.9000 0)
       (effects (font (size 1.27 1.27))))
-    (property "Footprint" "" (at 280.0000 270.8200 0)
+    (property "Footprint" "test-platform:R3" (at 280.0000 270.8200 0)
       (effects (font (size 1.27 1.27)) hide))
     (property "Datasheet" "" (at 280.0000 270.8200 0)
@@
     (property "Value" "10k" (at 280.0000 298.9800 0)
       (effects (font (size 1.27 1.27))))
-    (property "Footprint" "" (at 280.0000 293.9000 0)
+    (property "Footprint" "test-platform:R4" (at 280.0000 293.9000 0)
       (effects (font (size 1.27 1.27)) hide))
     (property "Datasheet" "" (at 280.0000 293.9000 0)
@@
     (property "Value" "10k" (at 280.0000 322.0600 0)
       (effects (font (size 1.27 1.27))))
-    (property "Footprint" "" (at 280.0000 316.9800 0)
+    (property "Footprint" "test-platform:R5" (at 280.0000 316.9800 0)
       (effects (font (size 1.27 1.27)) hide))
     (property "Datasheet" "" (at 280.0000 316.9800 0)
@@
     (property "Value" "10k" (at 280.0000 345.1400 0)
       (effects (font (size 1.27 1.27))))
-    (property "Footprint" "" (at 280.0000 340.0600 0)
+    (property "Footprint" "test-platform:R6" (at 280.0000 340.0600 0)
       (effects (font (size 1.27 1.27)) hide))
     (property "Datasheet" "" (at 280.0000 340.0600 0)
@@
     (property "Value" "220" (at 380.0000 32.6200 0)
       (effects (font (size 1.27 1.27))))
-    (property "Footprint" "" (at 380.0000 27.5400 0)
+    (property "Footprint" "test-platform:R7" (at 380.0000 27.5400 0)
       (effects (font (size 1.27 1.27)) hide))
     (property "Datasheet" "" (at 380.0000 27.5400 0)

Commit message: Removed PDF creation of test docs
Parts:
- removed M2: ADS1115_0x49, test-platform:M2, symbol test-platform:M2
- removed R1: LDR, test-platform:R1, symbol test-platform:R1
- removed R2: LDR, test-platform:R2, symbol test-platform:R2
- removed R3: LDR, test-platform:R3, symbol test-platform:R3
- removed R4: 10k, test-platform:R4, symbol test-platform:R4
- removed R5: 10k, test-platform:R5, symbol test-platform:R5
- removed R6: 10k, test-platform:R6, symbol test-platform:R6
- added D1: centre_LED, test-platform:D1, symbol test-platform:D1
- added R8: 330, test-platform:R8, symbol test-platform:R8
- added SW1: CW_limit_switch, test-platform:SW1, symbol test-platform:SW1
- added SW2: CCW_limit_switch, test-platform:SW2, symbol test-platform:SW2
- added U6: MCP23017, test-platform:U6, symbol test-platform:U6
Connections:
- net +3V3: now also SW1.2, SW2.2, U6.15 (A0), U6.18 (RESET), U6.9 (VDD)
- net EXP_IN1: now also U6.21 (GPA0); no longer U1.21 (GPA0)
- net EXP_IN2: now also U6.22 (GPA1); no longer U1.22 (GPA1)
- net EXP_IN3: now also U6.23 (GPA2); no longer U1.23 (GPA2)
- net EXP_IN4: now also U6.24 (GPA3); no longer U1.24 (GPA3)
- net GND: now also D1.K, U6.10 (VSS), U6.16 (A1), U6.17 (A2)
- net I2C_SCL: now also U6.12 (SCL)
- net I2C_SDA: now also U6.13 (SDA)
- net LCD_D5: now also SW1.1
- net LCD_D6: now also SW2.1
- net LED_CTRL: now reaches J1.35 (GPIO19)
- net LED_CTRL: now also R8.1
- new net LED_ANODE: D1.A, R8.2
Other:
- moved on the sheet: M1, M3, M4, R7, U2, U3, U4, U5
