File: docs/test-platform/kicad/test-platform.kicad_sch (KiCad schematic)
At the start: 22 parts, among them J1 Raspberry_Pi_40pin, M1 ADS1115_0x48, M3 DS3231_ZS042, M4 BMP180, M5 SSD1306_OLED, M6 BSS138_LLC, M7 ULN2003_28BYJ48, M8 LCD_HD44780, SW1 CW_limit_switch, SW2 CCW_limit_switch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

Commit message: test-platform singularity project updates
Connections:
- net EXP_LB4: now also U1.4 (GPB3); no longer U1.5 (GPB4)
- net EXP_LB5: now also U1.3 (GPB2); no longer U1.6 (GPB5)
- net EXP_LB6: now also U1.2 (GPB1); no longer U1.7 (GPB6)
- net EXP_LB7: now also U1.1 (GPB0); no longer U1.8 (GPB7)
- net EXP_LB0: now reaches U1.21 (GPA0)
- net EXP_LB0: now also U1.8 (GPB7)
- net EXP_LB1: now reaches U1.22 (GPA1)
- net EXP_LB1: now also U1.7 (GPB6)
- net EXP_LB2: now reaches U1.23 (GPA2)
- net EXP_LB2: now also U1.6 (GPB5)
- net EXP_LB3: now reaches U1.24 (GPA3)
- net EXP_LB3: now also U1.5 (GPB4)
Changed lines of the file:
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@@
     (effects (font (size 1.27 1.27)) (justify right))
+)
+  (label "EXP_LB0" (at 164.7600 52.9400 0)
+    (effects (font (size 1.27 1.27)) (justify right))
+)
+  (label "EXP_LB1" (at 164.7600 55.4800 0)
+    (effects (font (size 1.27 1.27)) (justify right))
+)
+  (label "EXP_LB2" (at 164.7600 58.0200 0)
+    (effects (font (size 1.27 1.27)) (justify right))
+)
+  (label "EXP_LB3" (at 195.2400 27.5400 0)
+    (effects (font (size 1.27 1.27)) (justify left))
 )
   (label "EXP_LB4" (at 195.2400 30.0800 0)
@@
     (effects (font (size 1.27 1.27)) (justify left))
 )
-  (label "EXP_LB4" (at 195.2400 50.4000 0)
+  (label "EXP_LB7" (at 195.2400 40.2400 0)
     (effects (font (size 1.27 1.27)) (justify left))
 )
-  (label "EXP_LB5" (at 195.2400 52.9400 0)
+  (label "EXP_LB6" (at 195.2400 42.7800 0)
     (effects (font (size 1.27 1.27)) (justify left))
 )
-  (label "EXP_LB6" (at 195.2400 55.4800 0)
+  (label "EXP_LB5" (at 195.2400 45.3200 0)
     (effects (font (size 1.27 1.27)) (justify left))
 )
-  (label "EXP_LB7" (at 195.2400 58.0200 0)
+  (label "EXP_LB4" (at 195.2400 47.8600 0)
     (effects (font (size 1.27 1.27)) (justify left))
 )
+  (label "EXP_LB3" (at 195.2400 50.4000 0)
+    (effects (font (size 1.27 1.27)) (justify left))
+)
+  (label "EXP_LB2" (at 195.2400 52.9400 0)
+    (effects (font (size 1.27 1.27)) (justify left))
+)
+  (label "EXP_LB1" (at 195.2400 55.4800 0)
+    (effects (font (size 1.27 1.27)) (justify left))
+)
+  (label "EXP_LB0" (at 195.2400 58.0200 0)
+    (effects (font (size 1.27 1.27)) (justify left))
+)
