File: docs/test-platform/kicad/rpi-wiringpi-unit-test-platform-board-4/rpi-wiringpi-unit-test-platform-board-4.kicad_sch (KiCad schematic)
At the start: 8 parts, among them J1 JST_IN_PWR, J2 JST_IN_I2C, M1 DS3231_0x68+AT24C32_0x57, M2 BMP180_0x77, M3 SSD1306_0x3c, SW1 SW_DIP_x01

Commit message: Updated boards
Parts:
- removed J1: JST_IN_PWR, rpi-wiringpi-unit-test-platform-board-4:J1, symbol rpi-wiringpi-unit-test-platform-board-4:J1
- removed J2: JST_IN_I2C, rpi-wiringpi-unit-test-platform-board-4:J2, symbol rpi-wiringpi-unit-test-platform-board-4:J2
- removed M2: BMP180_0x77, rpi-wiringpi-unit-test-platform-board-4:M2, symbol rpi-wiringpi-unit-test-platform-board-4:M2
- removed M3: SSD1306_0x3c, rpi-wiringpi-unit-test-platform-board-4:M3, symbol rpi-wiringpi-unit-test-platform-board-4:M3
- added C1: 10µf, Capacitor_THT:CP_Radial_D5.0mm_P2.50mm, symbol Device:C_Polarized
- added J3: JST_IN, Connector_JST:JST_XH_B5B-XH-A_1x05_P2.50mm_Vertical, symbol Connector:Conn_01x05_Pin
- added M2: BMP180, RPi:BMP180, symbol RPi:BMP180
- added OLED1: SSD1306_128_64, RPi:OLED_SSD_1306_128_64, symbol RPi:OLED_SSD1306_128_64
- D1: value LED -> LED_BOARD_CONN; footprint rpi-wiringpi-unit-test-platform-board-4:D1 -> LED_THT:LED_D5.0mm; symbol rpi-wiringpi-unit-test-platform-board-4:D1 -> Device:LED
- R1: value R -> 330; footprint rpi-wiringpi-unit-test-platform-board-4:R1 -> Resistor_THT:R_Axial_DIN0207_L6.3mm_D2.5mm_P7.62mm_Horizontal
Connections:
- net +3V3: now also SW1.2, C1.1, J3.1 (Pin_1), J3.3 (Pin_3), M2.2 (3V3), OLED1.2 (VCC)
- net GND: now also R1.1, C1.2, J3.2 (Pin_2), M2.3 (GND), OLED1.1 (GND)
- net I2C_SCL: now also J3.5 (Pin_5), M2.4 (SCL), OLED1.3 (SCL)
- net I2C_SDA: now also J3.4 (Pin_4), M2.5 (SDA), OLED1.4 (SDA)
- net at R1.2: now also D1.1 (K)
- net at SW1.1: now also D1.2 (A)
- no-connect marks 0 -> 3
Other:
- moved on the sheet: M1, R1, SW1

Commit message: Finalize board 4 hardware
Parts:
- M1: footprint rpi-wiringpi-unit-test-platform-board-4:M1 -> RPi:DS3231
- SW1: footprint rpi-wiringpi-unit-test-platform-board-4:SW1 -> Button_Switch_SMD:SW_DIP_SPSTx01_Slide_6.7x4.1mm_W6.73mm_P2.54mm_LowProfile_JPin
Changed lines of the file:
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@@
 			)
 		)
-		(property "Footprint" "rpi-wiringpi-unit-test-platform-board-4:M1"
+		(property "Footprint" "RPi:DS3231"
 			(at 72.39 115.57 0)
 			(hide yes)
@@
 			)
 		)
-		(property "Footprint" "rpi-wiringpi-unit-test-platform-board-4:SW1"
+		(property "Footprint" "Button_Switch_SMD:SW_DIP_SPSTx01_Slide_6.7x4.1mm_W6.73mm_P2.54mm_LowProfile_JPin"
 			(at 95.25 140.97 0)
 			(hide yes)

Commit message: Finish boards
Parts:
- removed M1: DS3231_0x68+AT24C32_0x57, RPi:DS3231, symbol rpi-wiringpi-unit-test-platform-board-4:M1
- added M1: DS3231_0x68+AT24C32_0x57, RPi:DS3231, symbol RPi:DS3231
Connections:
- net +3V3: now also M1.2 (VCC)
- net GND: now also M1.1 (GND)
- net I2C_SCL: now also M1.4 (SCL)
- net I2C_SDA: now also M1.3 (SDA)
Changed lines of the file:
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@@
 	(generator_version "10.0")
 	(paper "USLetter" portrait)
+	(title_block
+		(date "2026-07-06")
+		(rev "2")
+	)
 	(junction
 		(at 99.06 87.63)
@@
 	)
 	(junction
+		(at 91.44 102.87)
+		(diameter 0)
+		(color 0 0 0 0)
+	)
+	(junction
 		(at 50.8 118.11)
 		(diameter 0)
@@
 	)
 	(junction
-		(at 50.8 102.87)
-		(diameter 0)
-		(color 0 0 0 0)
-	)
-	(junction
 		(at 43.18 30.48)
 		(diameter 0)
@@
 	)
 	(no_connect
-		(at 87.63 118.11)
+		(at 82.55 118.11)
 	)
 	(no_connect
@@
 	)
 	(no_connect
-		(at 87.63 115.57)
+		(at 82.55 115.57)
 	)
 	(wire
@@
 	(wire
 		(pts
-			(xy 50.8 48.26) (xy 50.8 102.87)
+			(xy 50.8 48.26) (xy 50.8 118.11)
 		)
 		(stroke
@@
 	(wire
 		(pts
+			(xy 74.93 102.87) (xy 91.44 102.87)
+		)
+		(stroke
+			(width 0)
+			(type default)
+		)
+	)
+	(wire
+		(pts
 			(xy 62.23 48.26) (xy 74.93 48.26)
 		)
@@
 	(wire
 		(pts
-			(xy 45.72 115.57) (xy 57.15 115.57)
+			(xy 45.72 115.57) (xy 60.96 115.57)
 		)
 		(stroke
@@
 	(wire
 		(pts
-			(xy 50.8 102.87) (xy 50.8 118.11)
-		)
-		(stroke
-			(width 0)
-			(type default)
-		)
-	)
-	(wire
-		(pts
 			(xy 74.93 48.26) (xy 74.93 64.77)
 		)
@@
 	(wire
 		(pts
+			(xy 82.55 113.03) (xy 99.06 113.03)
+		)
+		(stroke
+			(width 0)
+			(type default)
+		)
+	)
+	(wire
+		(pts
 			(xy 38.1 34.29) (xy 43.18 34.29)
 		)
@@
 	(wire
 		(pts
-			(xy 91.44 62.23) (xy 91.44 129.54)
+			(xy 57.15 113.03) (xy 60.96 113.03)
+		)
+		(stroke
+			(width 0)
+			(type default)
+		)
+	)
+	(wire
+		(pts
+			(xy 91.44 62.23) (xy 91.44 102.87)
 		)
 		(stroke
@@
 	(wire
 		(pts
-			(xy 87.63 113.03) (xy 99.06 113.03)
+			(xy 91.44 102.87) (xy 91.44 129.54)
 		)
 		(stroke
@@
 	(wire
 		(pts
-			(xy 57.15 118.11) (xy 50.8 118.11)
+			(xy 50.8 118.11) (xy 60.96 118.11)
 		)
 		(stroke
@@
 		(pts
 			(xy 54.61 105.41) (xy 57.15 105.41)
-		)
-		(stroke
-			(width 0)
-			(type default)
-		)
-	)
-	(wire
-		(pts
-			(xy 74.93 102.87) (xy 50.8 102.87)
 		)
 		(stroke
@@
 		)
 	)
+	(label "I2C_SCL"
+		(at 85.09 113.03 0)
+		(effects
+			(font
+				(size 1.27 1.27)
+			)
+			(justify left bottom)
+		)
+	)
 	(label "I2C_SDA"
 		(at 50.8 69.85 0)
+		(effects
+			(font
+				(size 1.27 1.27)
+			)
+			(justify left bottom)
+		)
+	)
+	(label "I2C_SDA"
+		(at 52.07 118.11 0)
 		(effects
 			(font
@@
 	)
 	(symbol
-		(lib_name "OLED_SSD1306_128_64_1")
 		(lib_id "RPi:OLED_SSD1306_128_64")
 		(at 71.12 91.44 0)
@@
 				(path "/dc869679-2405-5a19-9d54-909a37e7887e"
 					(reference "OLED1")
+					(unit 1)
+				)
+			)
+		)
+	)
+	(symbol
+		(lib_id "RPi:DS3231")
+		(at 71.12 115.57 0)
+		(unit 1)
+		(body_style 1)
+		(exclude_from_sim no)
+		(in_bom yes)
+		(on_board yes)
+		(in_pos_files yes)
+		(dnp no)
+		(property "Reference" "M1"
+			(at 71.755 105.41 0)
+			(show_name no)
+			(do_not_autoplace no)
+			(effects
+				(font
+					(size 1.27 1.27)
+				)
+			)
+		)
+		(property "Value" "DS3231_0x68+AT24C32_0x57"
+			(at 71.628 125.476 0)
+			(show_name no)
+			(do_not_autoplace no)
+			(effects
+				(font
+					(size 1.27 1.27)
+				)
+			)
+		)
+		(property "Footprint" "RPi:DS3231"
+			(at 71.12 115.57 0)
+			(hide yes)
+			(show_name no)
+			(do_not_autoplace no)
+			(effects
+				(font
+					(size 1.27 1.27)
+				)
+			)
+		)
+		(property "Datasheet" ""
+			(at 71.12 115.57 0)
+			(hide yes)
+			(show_name no)
+			(do_not_autoplace no)
+			(effects
+				(font
+					(size 1.27 1.27)
+				)
+			)
+		)
+		(property "Description" ""
+			(at 71.12 115.57 0)
+			(hide yes)
+			(show_name no)
+			(do_not_autoplace no)
+			(effects
+				(font
+					(size 1.27 1.27)
+				)
+			)
+		)
+		(pin "2"
+		)
+		(pin "6"
+		)
+		(pin "1"
+		)
+		(pin "3"
+		)
+		(pin "4"
+		)
+		(pin "5"
+		)
+		(instances
+			(project "rpi-wiringpi-unit-test-platform-board-4"
+				(path "/dc869679-2405-5a19-9d54-909a37e7887e"
+					(reference "M1")
 					(unit 1)
 				)
@@
 					(unit 1)
 				)
-			)
-		)
-	)
-	(symbol
-		(lib_id "rpi-wiringpi-unit-test-platform-board-4:M1")
-		(at 72.39 115.57 0)
-		(unit 1)
-		(body_style 1)
-		(exclude_from_sim no)
-		(in_bom yes)
-		(on_board yes)
-		(in_pos_files yes)
-		(dnp no)
-		(property "Reference" "M1"
-			(at 72.39 107.95 0)
-			(show_name no)
-			(do_not_autoplace no)
-			(effects
-				(font
-					(size 1.27 1.27)
-				)
-			)
-		)
-		(property "Value" "DS3231_0x68+AT24C32_0x57"
-			(at 72.39 123.19 0)
-			(show_name no)
-			(do_not_autoplace no)
-			(effects
-				(font
-					(size 1.27 1.27)
-				)
-			)
-		)
-		(property "Footprint" "RPi:DS3231"
-			(at 72.39 115.57 0)
-			(hide yes)
-			(show_name no)
-			(do_not_autoplace no)
-			(effects
-				(font
-					(size 1.27 1.27)
-				)
-			)
-		)
-		(property "Datasheet" ""
-			(at 72.39 115.57 0)
-			(hide yes)
-			(show_name no)
-			(do_not_autoplace no)
-			(effects
-				(font
-					(size 1.27 1.27)
-				)
-			)
-		)
-		(property "Description" ""
-			(at 72.39 115.57 0)
-			(show_name no)
-			(do_not_autoplace no)
-			(effects
-				(font
-					(size 1.27 1.27)
-				)
-			)
-		)
-		(pin "1"
-		)
-		(pin "2"
-		)
-		(pin "3"
-		)
-		(pin "4"
-		)
-		(pin "5"
-		)
-		(pin "6"
-		)
-		(instances
-			(project "rpi-wiringpi-unit-test-platform-board-4"
-				(path "/dc869679-2405-5a19-9d54-909a37e7887e"
-					(reference "M1")
-					(unit 1)
-				)

Commit message: Cleanup of PCBs/schematics
Parts:
- removed SW1: SW_DIP_x01, Button_Switch_SMD:SW_DIP_SPSTx01_Slide_6.7x4.1mm_W6.73mm_P2.54mm_LowProfile_JPin, symbol rpi-wiringpi-unit-test-platform-board-4:SW1
- added SW1: SW_DIP_x01, Button_Switch_THT:SW_DIP_SPSTx01_Slide_9.78x4.72mm_W7.62mm_P2.54mm, symbol Switch:SW_DIP_x01
Connections:
- net +3V3: now also SW1.2
- net at D1.2 (A): now also SW1.1
Changed lines of the file:
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@@
+	(wire
+		(pts
+			(xy 100.33 140.97) (xy 110.49 140.97)
+		)
+		(stroke
+			(width 0)
+			(type default)
+		)
+	)
 	(wire
 		(pts
@@
 	(wire
 		(pts
-			(xy 74.93 140.97) (xy 80.01 140.97)
+			(xy 74.93 140.97) (xy 85.09 140.97)
 		)
 		(stroke
@@
 	)
 	(symbol
-		(lib_id "rpi-wiringpi-unit-test-platform-board-4:SW1")
-		(at 95.25 140.97 0)
-		(unit 1)
-		(body_style 1)
-		(exclude_from_sim no)
-		(in_bom yes)
-		(on_board yes)
-		(in_pos_files yes)
-		(dnp no)
-		(property "Reference" "SW1"
-			(at 95.25 135.89 0)
-			(show_name no)
-			(do_not_autoplace no)
-			(effects
-				(font
-					(size 1.27 1.27)
-				)
-			)
-		)
-		(property "Value" "SW_DIP_x01"
-			(at 95.25 146.05 0)
-			(show_name no)
-			(do_not_autoplace no)
-			(effects
-				(font
-					(size 1.27 1.27)
-				)
-			)
-		)
-		(property "Footprint" "Button_Switch_SMD:SW_DIP_SPSTx01_Slide_6.7x4.1mm_W6.73mm_P2.54mm_LowProfile_JPin"
-			(at 95.25 140.97 0)
-			(hide yes)
-			(show_name no)
-			(do_not_autoplace no)
-			(effects
-				(font
-					(size 1.27 1.27)
-				)
-			)
-		)
-		(property "Datasheet" ""
-			(at 95.25 140.97 0)
-			(hide yes)
-			(show_name no)
-			(do_not_autoplace no)
-			(effects
-				(font
-					(size 1.27 1.27)
-				)
-			)
-		)
-		(property "Description" ""
-			(at 95.25 140.97 0)
-			(show_name no)
-			(do_not_autoplace no)
-			(effects
-				(font
-					(size 1.27 1.27)
-				)
-			)
-		)
-		(pin "1"
-		)
-		(pin "2"
-		)
-		(instances
-			(project "rpi-wiringpi-unit-test-platform-board-4"
-				(path "/dc869679-2405-5a19-9d54-909a37e7887e"
-					(reference "SW1")
-					(unit 1)
-				)
-			)
-		)
-	)
-	(symbol
 		(lib_id "Device:C_Polarized")
 		(at 44.45 43.18 270)
@@
 					(unit 1)
 				)
+			)
+		)
+	)
+	(symbol
+		(lib_id "Switch:SW_DIP_x01")
+		(at 92.71 140.97 0)
+		(unit 1)
+		(body_style 1)
+		(exclude_from_sim no)
+		(in_bom yes)
+		(on_board yes)
+		(in_pos_files yes)
+		(dnp no)
+		(fields_autoplaced yes)
+		(property "Reference" "SW1"
+			(at 92.71 133.35 0)
+			(show_name no)
+			(do_not_autoplace no)
+			(effects
+				(font
+					(size 1.27 1.27)
+				)
+			)
+		)
+		(property "Value" "SW_DIP_x01"
+			(at 92.71 135.89 0)
+			(show_name no)
+			(do_not_autoplace no)
+			(effects
+				(font
+					(size 1.27 1.27)
+				)
+			)
+		)
+		(property "Footprint" "Button_Switch_THT:SW_DIP_SPSTx01_Slide_9.78x4.72mm_W7.62mm_P2.54mm"
+			(at 92.71 140.97 0)
+			(hide yes)
+			(show_name no)
+			(do_not_autoplace no)
+			(effects
+				(font
+					(size 1.27 1.27)
+				)
+			)
+		)
+		(property "Datasheet" ""
+			(at 92.71 140.97 0)
+			(hide yes)
+			(show_name no)
+			(do_not_autoplace no)
+			(effects
+				(font
+					(size 1.27 1.27)
+				)
+			)
+		)
+		(property "Description" "1x DIP Switch, Single Pole Single Throw (SPST) switch, small symbol"
+			(at 92.71 140.97 0)
+			(hide yes)
+			(show_name no)
+			(do_not_autoplace no)
+			(effects
+				(font
+					(size 1.27 1.27)
+				)
+			)
+		)
+		(pin "2"
+		)
+		(pin "1"
+		)
+		(instances
+			(project "rpi-wiringpi-unit-test-platform-board-4"
+				(path "/dc869679-2405-5a19-9d54-909a37e7887e"
+					(reference "SW1")
+					(unit 1)
+				)
