File: docs/test-platform/kicad/rpi-wiringpi-unit-test-platform-board-5/rpi-wiringpi-unit-test-platform-board-5.kicad_sch (KiCad schematic)
At the start: 9 parts, among them J1 JST_IN_PWR, J2 JST_IN_SIG, J3 JST_IN_LCD, J4 JST_OUT_I2C5V, U1 LVLSHIFT_BOB12009

Commit message: Work on test board 5
Parts:
- removed JP1: UART_LOOP, rpi-wiringpi-unit-test-platform-board-5:JP1, symbol rpi-wiringpi-unit-test-platform-board-5:JP1
- added SW1: SW_DIP_x01, Button_Switch_THT:SW_DIP_SPSTx01_Slide_9.78x4.72mm_W7.62mm_P2.54mm, symbol Switch:SW_DIP_x01
Connections:
- net UART_RX: now also SW1.2
- net UART_TX: now also SW1.1
- no-connect marks 0 -> 8
Other:
- moved on the sheet: J1, J2, J3, J4, LCD1, R1, RV1, U1

Commit message: Finished KiCAD test board 5
Parts:
- removed R1: 220, rpi-wiringpi-unit-test-platform-board-5:R1, symbol rpi-wiringpi-unit-test-platform-board-5:R1
- removed SW1: SW_DIP_x01, Button_Switch_THT:SW_DIP_SPSTx01_Slide_9.78x4.72mm_W7.62mm_P2.54mm, symbol Switch:SW_DIP_x01
- added D1: LED_BOARD_CONN, LED_THT:LED_D5.0mm, symbol Device:LED
- added R1: 330, Resistor_THT:R_Axial_DIN0207_L6.3mm_D2.5mm_P7.62mm_Horizontal, symbol Device:R
- added SW1: SW_DIP_x03, Button_Switch_THT:SW_DIP_SPSTx03_Slide_9.78x9.8mm_W7.62mm_P2.54mm, symbol Switch:SW_DIP_x03
- J4: value JST_OUT_I2C5V -> JST_OUT_ARDUINO
- U1: value LVLSHIFT_BOB12009 -> LVLSHIFT
Connections:
- net +3V3: now also SW1.3
- net +5V: now also SW1.5
- net GND: now also R1.2
- net LCD_BL_A: now also SW1.2
- net UART_RX: now also SW1.1
- net UART_TX: now also SW1.6
- new net: D1.2 (A), SW1.4
- new net: D1.1 (K), R1.1

Commit message: Finalization work on test board 5
Parts:
- LCD1: value HD44780_20x4 -> HD44780_20x2
- RV1: value 10k -> LCD_DIMMER
Changed lines of the file:
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@@
 			)
 		)
-		(property "Value" "10k"
+		(property "Value" "LCD_DIMMER"
 			(at 41.91 77.47 0)
 			(show_name no)
@@
 			)
 		)
-		(property "Value" "HD44780_20x4"
+		(property "Value" "HD44780_20x2"
 			(at 38.1 48.26 0)
 			(show_name no)

Commit message: Added decoupling caps
Parts:
- added C1, C2: 0.1 µF, Capacitor_THT:C_Disc_D5.0mm_W2.5mm_P2.50mm, symbol Device:C
- added C3: 10 µF, Capacitor_THT:CP_Radial_D5.0mm_P2.50mm, symbol Device:C_Polarized_Small_US
Connections:
- net +3V3: now also C1.1, C2.1, C3.1
- net GND: now also C1.2, C2.2, C3.2
