File: docs/test-platform/kicad/rpi-wiringpi-unit-test-platform-board-5/rpi-wiringpi-unit-test-platform-board-5.kicad_pcb (KiCad board)
At the start: 2 copper layers, 95.2 x 49.5 mm, 19 parts, among them J1 JST_IN_PWR, J2 JST_IN_SIG, J3 JST_IN_LCD, J4 JST_OUT_ARDUINO, M1 Logic_Lvl_Shifter, SW1 SW_CTRL, U1 LCD_HD44780

Commit message: Fix capacitor conflicts related to datasheets; add cap conflict checks to build
Other:
- board text added: "Perl RPi::WiringPi test platform Board 5 Revision: ${REVISION} Steve Bertrand ${CURRENT_DATE}"
- board text removed: "Perl RPi::WiringPi test platform Board 5 Revision: ${REVISION} Steve Bertrand 20260623"
Changed lines of the file:
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@@
 	(title_block
 		(date "2026-06-23")
-		(rev "1")
+		(rev "2")
 	)
 	(layers
@@
 		)
 	)
-	(gr_text "Perl RPi::WiringPi test platform Board 5\nRevision: ${REVISION}\nSteve Bertrand\n20260623"
+	(gr_text "Perl RPi::WiringPi test platform Board 5\nRevision: ${REVISION}\nSteve Bertrand\n${CURRENT_DATE}"
 		(at 129.54 104.14 0)
 		(layer "F.SilkS")
@@
 	)
 	(segment
+		(start 152.4 83.82)
+		(end 153.67 82.55)
+		(width 0.25)
+		(layer "F.Cu")
+		(net "/LED_BRD_CONN")
+	)
+	(segment
+		(start 139.7 83.82)
+		(end 152.4 83.82)
+		(width 0.25)
+		(layer "F.Cu")
+		(net "/LED_BRD_CONN")
+	)
+	(segment
 		(start 146.047208 92.71)
 		(end 143.51 92.71)
@@
 		(net "Net-(D1-K)")
 	)
-	(segment
-		(start 99.205 92.565)
-		(end 113.215 92.565)
-		(width 0.4)
-		(layer "F.Cu")
-		(net "/LCD_V0")
-	)
-	(segment
-		(start 113.215 92.565)
-		(end 120.69 85.09)
-		(width 0.4)
-		(layer "F.Cu")
-		(net "/LCD_V0")
-	)
-	(segment
-		(start 93.726 98.044)
-		(end 99.205 92.565)
-		(width 0.4)
-		(layer "F.Cu")
-		(net "/LCD_V0")
-	)
 	(via
 		(at 130.81 73.66)
@@
 	)
 	(segment
+		(start 99.205 92.565)
+		(end 113.215 92.565)
+		(width 0.4)
+		(layer "F.Cu")
+		(net "/LCD_V0")
+	)
+	(segment
+		(start 113.215 92.565)
+		(end 120.69 85.09)
+		(width 0.4)
+		(layer "F.Cu")
+		(net "/LCD_V0")
+	)
+	(segment
+		(start 93.726 98.044)
+		(end 99.205 92.565)
+		(width 0.4)
+		(layer "F.Cu")
+		(net "/LCD_V0")
+	)
+	(segment
 		(start 148.910991 68.58)
 		(end 148.63 68.58)
@@
 	)
 	(segment
+		(start 129.54 92.71)
+		(end 135.89 92.71)
+		(width 0.25)
+		(layer "B.Cu")
+		(net "Net-(U1-BL-A(+))")
+	)
+	(segment
+		(start 124.206 98.044)
+		(end 129.54 92.71)
+		(width 0.25)
+		(layer "B.Cu")
+		(net "Net-(U1-BL-A(+))")
+	)
+	(segment
 		(start 93.98 76.207)
 		(end 93.98 82.55)
@@
 		(net "/I2C_SCL")
 	)
-	(segment
-		(start 152.4 83.82)
-		(end 153.67 82.55)
-		(width 0.25)
-		(layer "F.Cu")
-		(net "/LED_BRD_CONN")
-	)
-	(segment
-		(start 139.7 83.82)
-		(end 152.4 83.82)
-		(width 0.25)
-		(layer "F.Cu")
-		(net "/LED_BRD_CONN")
-	)
-	(segment
-		(start 129.54 92.71)
-		(end 135.89 92.71)
-		(width 0.25)
-		(layer "B.Cu")
-		(net "Net-(U1-BL-A(+))")
-	)
-	(segment
-		(start 124.206 98.044)
-		(end 129.54 92.71)
-		(width 0.25)
-		(layer "B.Cu")
-		(net "Net-(U1-BL-A(+))")
-	)
 	(zone
