File: docs/test-platform/kicad/rpi-wiringpi-unit-test-platform-board-3/rpi-wiringpi-unit-test-platform-board-3.kicad_pcb (KiCad board)
At the start: 2 copper layers, 91.4 x 67.9 mm, 28 parts, among them J1 JST_IN_PWR, J2 JST_IN_SIG, J3 JST_OUT_PWR, J4 JST_OUT_SW, J5 JST_OUT_COIL, J6 JST_IO_A4_7, J7 JST_IO_B0_3, J8 JST_IO_B4_7, SW1 LED_SW, U1 MCP23017_0x20, U2 MCP23017_0x21

Commit message: Massive cleanup (build_testing, fritzing etc)
Parts:
- renumbered R7 to R5, R8 to R6
Changed lines of the file:
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@@
 		(descr "Resistor, Axial_DIN0207 series, Axial, Horizontal, pin pitch=7.62mm, 0.25W = 1/4W, length*diameter=6.3*2.5mm^2, http://cdn-reichelt.de/documents/datenblatt/B400/1_4W%23YAG.pdf")
 		(tags "Resistor Axial_DIN0207 series Axial Horizontal pin pitch 7.62mm 0.25W = 1/4W length 6.3mm diameter 2.5mm")
-		(property "Reference" "R8"
+		(property "Reference" "R6"
 			(at 0 -2.54 180)
 			(layer "F.SilkS")
@@
 		(descr "Resistor, Axial_DIN0207 series, Axial, Horizontal, pin pitch=7.62mm, 0.25W = 1/4W, length*diameter=6.3*2.5mm^2, http://cdn-reichelt.de/documents/datenblatt/B400/1_4W%23YAG.pdf")
 		(tags "Resistor Axial_DIN0207 series Axial Horizontal pin pitch 7.62mm 0.25W = 1/4W length 6.3mm diameter 2.5mm")
-		(property "Reference" "R7"
+		(property "Reference" "R5"
 			(at 0 -2.54 0)
 			(layer "F.SilkS")
