File: docs/test-platform/kicad/rpi-wiringpi-unit-test-platform-board-2/rpi-wiringpi-unit-test-platform-board-2.kicad_sch (KiCad schematic)
At the start: 22 parts, among them J1 IN_PWR, J2 IN_SIGNAL, J3 IN_CS_SHIFTREG, J4 OUT_SERVO, J5 OUT_SERVO_SIG, SW1 SW_BOARD_CONN_LED, U1 MCP3008, U2 MCP4922, U3 MCP42010, U4 ADS1115, U5 74HC595

Commit message: Fix capacitor conflicts related to datasheets; add cap conflict checks to build
Parts:
- C1: renamed from C5; KiLib_Generator (none) -> capacitor/THT/other
- C2, C3, C4, C6, C7, C8, C9: KiLib_Generator (none) -> capacitor/THT/other
- C5: renamed from C1; value 0.1µf -> 1µf; KiLib_Generator (none) -> capacitor/THT/other
- D1: KiLib_Generator (none) -> LED/THT
- J1, J2, J3, J4, J5: KiLib_Generator (none) -> connector/JST
- R1: KiLib_Generator (none) -> resistor/THT
- SW1: KiLib_Generator (none) -> button_switch/DIP
- U1, U2, U3, U5: KiLib_Generator (none) -> package/DIP/legacy
Changed lines of the file:
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@@
 	(title_block
 		(date "2026-07-22")
-		(rev "4")
+		(rev "5")
 	)
 	(junction
@@
 			)
 		)
+		(property "KiLib_Generator" "connector/JST"
+			(at 198.12 128.27 0)
+			(hide yes)
+			(show_name no)
+			(do_not_autoplace no)
+			(effects
+				(font
+					(size 1.27 1.27)
+				)
+			)
+		)
 		(pin "6"
 		)
@@
 			)
 		)
+		(property "KiLib_Generator" "capacitor/THT/other"
+			(at 217.17 45.72 0)
+			(hide yes)
+			(show_name no)
+			(do_not_autoplace no)
+			(effects
+				(font
+					(size 1.27 1.27)
+				)
+			)
+		)
 		(pin "1"
 		)
@@
 			)
 		)
+		(property "KiLib_Generator" "capacitor/THT/other"
+			(at 30.48 142.24 0)
+			(hide yes)
+			(show_name no)
+			(do_not_autoplace no)
+			(effects
+				(font
+					(size 1.27 1.27)
+				)
+			)
+		)
 		(pin "1"
 		)
@@
 			)
 		)
+		(property "KiLib_Generator" "connector/JST"
+			(at 198.12 96.52 0)
+			(hide yes)
+			(show_name no)
+			(do_not_autoplace no)
+			(effects
+				(font
+					(size 1.27 1.27)
+				)
+			)
+		)
 		(pin "6"
 		)
@@
 			)
 		)
+		(property "KiLib_Generator" "resistor/THT"
+			(at 168.91 46.99 0)
+			(hide yes)
+			(show_name no)
+			(do_not_autoplace no)
+			(effects
+				(font
+					(size 1.27 1.27)
+				)
+			)
+		)
 		(pin "2"
 		)
@@
 			)
 		)
+		(property "KiLib_Generator" "package/DIP/legacy"
+			(at 134.62 149.86 0)
+			(hide yes)
+			(show_name no)
+			(do_not_autoplace no)
+			(effects
+				(font
+					(size 1.27 1.27)
+				)
+			)
+		)
 		(pin "9"
 		)
@@
 			)
 		)
+		(property "KiLib_Generator" "package/DIP/legacy"
+			(at 134.62 95.25 0)
+			(hide yes)
+			(show_name no)
+			(do_not_autoplace no)
+			(effects
+				(font
+					(size 1.27 1.27)
+				)
+			)
+		)
 		(pin "2"
 		)
@@
 			)
 		)
+		(property "KiLib_Generator" "capacitor/THT/other"
+			(at 111.76 132.08 0)
+			(hide yes)
+			(show_name no)
+			(do_not_autoplace no)
+			(effects
+				(font
+					(size 1.27 1.27)
+				)
+			)
+		)
 		(pin "1"
 		)
@@
 			)
 		)
+		(property "KiLib_Generator" "connector/JST"
+			(at 96.52 110.49 0)
+			(hide yes)
+			(show_name no)
+			(do_not_autoplace no)
+			(effects
+				(font
+					(size 1.27 1.27)
+				)
+			)
+		)
 		(pin "1"
 		)
@@
 			)
 		)
+		(property "KiLib_Generator" "button_switch/DIP"
+			(at 199.39 34.29 0)
+			(hide yes)
+			(show_name no)
+			(do_not_autoplace no)
+			(effects
+				(font
+					(size 1.27 1.27)
+				)
+			)
+		)
 		(pin "1"
 		)
@@
 			)
 		)
+		(property "KiLib_Generator" "LED/THT"
+			(at 171.45 34.29 0)
+			(hide yes)
+			(show_name no)
+			(do_not_autoplace no)
+			(effects
+				(font
+					(size 1.27 1.27)
+				)
+			)
+		)
 		(pin "1"
 		)
@@
 		(dnp no)
 		(fields_autoplaced yes)
-		(property "Reference" "C1"
+		(property "Reference" "C5"
 			(at 165.1 73.6599 0)
 			(show_name no)
@@
 			)
 		)
-		(property "Value" "0.1µf"
+		(property "Value" "1µf"
 			(at 165.1 76.1999 0)
 			(show_name no)
@@
 			)
 		)
+		(property "KiLib_Generator" "capacitor/THT/other"
+			(at 161.29 74.93 0)
+			(hide yes)
+			(show_name no)
+			(do_not_autoplace no)
+			(effects
+				(font
+					(size 1.27 1.27)
+				)
+			)
+		)
 		(pin "1"
 		)
@@
 			(project "rpi-wiringpi-unit-test-platform-board-2"
 				(path "/7946ceed-5e50-51f0-9396-19e4533fa9f5"
-					(reference "C1")
+					(reference "C5")
 					(unit 1)
 				)
@@
 		(dnp no)
 		(fields_autoplaced yes)
-		(property "Reference" "C5"
+		(property "Reference" "C1"
 			(at 66.04 191.7699 0)
 			(show_name no)
@@
 			)
 		)
+		(property "KiLib_Generator" "capacitor/THT/other"
+			(at 62.23 193.04 0)
+			(hide yes)
+			(show_name no)
+			(do_not_autoplace no)
+			(effects
+				(font
+					(size 1.27 1.27)
+				)
+			)
+		)
 		(pin "1"
 		)
@@
 			(project "rpi-wiringpi-unit-test-platform-board-2"
 				(path "/7946ceed-5e50-51f0-9396-19e4533fa9f5"
-					(reference "C5")
+					(reference "C1")
 					(unit 1)
 				)
@@
 			)
 		)
+		(property "KiLib_Generator" "connector/JST"
+			(at 201.93 64.77 0)
+			(hide yes)
+			(show_name no)
+			(do_not_autoplace no)
+			(effects
+				(font
+					(size 1.27 1.27)
+				)
+			)
+		)
 		(pin "4"
 		)
@@
 			)
 		)
+		(property "KiLib_Generator" "capacitor/THT/other"
+			(at 220.98 149.86 0)
+			(hide yes)
+			(show_name no)
+			(do_not_autoplace no)
+			(effects
+				(font
+					(size 1.27 1.27)
+				)
+			)
+		)
 		(pin "1"
 		)
@@
 			)
 		)
+		(property "KiLib_Generator" "capacitor/THT/other"
+			(at 22.86 91.44 0)
+			(hide yes)
+			(show_name no)
+			(do_not_autoplace no)
+			(effects
+				(font
+					(size 1.27 1.27)
+				)
+			)
+		)
 		(pin "2"
 		)
@@
 			)
 		)
+		(property "KiLib_Generator" "capacitor/THT/other"
+			(at 105.41 132.08 0)
+			(hide yes)
+			(show_name no)
+			(do_not_autoplace no)
+			(effects
+				(font
+					(size 1.27 1.27)
+				)
+			)
+		)
 		(pin "1"
 		)
@@
 			)
 		)
+		(property "KiLib_Generator" "package/DIP/legacy"
+			(at 96.52 195.58 0)
+			(hide yes)
+			(show_name no)
+			(do_not_autoplace no)
+			(effects
+				(font
+					(size 1.27 1.27)
+				)
+			)
+		)
 		(pin "7"
 		)
@@
 			)
 		)
+		(property "KiLib_Generator" "capacitor/THT/other"
+			(at 212.09 149.86 0)
+			(hide yes)
+			(show_name no)
+			(do_not_autoplace no)
+			(effects
+				(font
+					(size 1.27 1.27)
+				)
+			)
+		)
 		(pin "1"
 		)
@@
 			)
 		)
+		(property "KiLib_Generator" "package/DIP/legacy"
+			(at 58.42 95.25 0)
+			(hide yes)
+			(show_name no)
+			(do_not_autoplace no)
+			(effects
+				(font
+					(size 1.27 1.27)
+				)
+			)
+		)
 		(pin "5"
 		)
@@
 			(at 201.93 157.48 0)
 			(hide yes)
+			(show_name no)
+			(do_not_autoplace no)
+			(effects
+				(font
+					(size 1.27 1.27)
+				)
+			)
+		)
+		(property "KiLib_Generator" "connector/JST"
+			(at 201.93 157.48 0)
+			(hide yes)

Commit message: Change footprint of cap to tantalum for the mcp4922
Parts:
- C8: footprint Capacitor_THT:CP_Radial_D5.0mm_P2.50mm -> Capacitor_THT:CP_Radial_Tantal_D5.0mm_P2.50mm
Changed lines of the file:
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@@
 			)
 		)
-		(property "Footprint" "Capacitor_THT:CP_Radial_D5.0mm_P2.50mm"
+		(property "Footprint" "Capacitor_THT:CP_Radial_Tantal_D5.0mm_P2.50mm"
 			(at 106.3752 135.89 0)
 			(hide yes)

Commit message: Re-footprint caps
Parts:
- C6: footprint Capacitor_THT:CP_Radial_D6.3mm_P2.50mm -> Capacitor_THT:CP_Radial_D5.0mm_P2.50mm
- C7: footprint Capacitor_THT:CP_Radial_D6.3mm_P2.50mm -> Capacitor_THT:CP_Radial_D8.0mm_P2.50mm
Changed lines of the file:
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@@
 			)
 		)
-		(property "Footprint" "Capacitor_THT:CP_Radial_D6.3mm_P2.50mm"
+		(property "Footprint" "Capacitor_THT:CP_Radial_D5.0mm_P2.50mm"
 			(at 218.44 49.53 0)
 			(hide yes)
@@
 			)
 		)
-		(property "Footprint" "Capacitor_THT:CP_Radial_D6.3mm_P2.50mm"
+		(property "Footprint" "Capacitor_THT:CP_Radial_D8.0mm_P2.50mm"
 			(at 222.25 153.67 0)
 			(hide yes)

Commit message: Cleanup tracing
Parts:
- D1: value LED_BOARD_CONN -> LED_BRD_CONN_SIG
- SW1: value SW_BOARD_CONN_LED -> SW_BRD_CONN_SIG
Connections:
- net +3V3: no longer J1.4 (Pin_4), SW1.2
- new net CONN_SIG: J1.4 (Pin_4), SW1.2
Other:
- moved on the sheet: R1
Changed lines of the file:
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@@
 	)
 	(junction
-		(at 187.96 64.77)
-		(diameter 0)
-		(color 0 0 0 0)
-	)
-	(junction
 		(at 134.62 137.16)
 		(diameter 0)
@@
 	)
 	(junction
-		(at 207.01 69.85)
-		(diameter 0)
-		(color 0 0 0 0)
-	)
-	(junction
 		(at 207.01 67.31)
 		(diameter 0)
@@
 	)
 	(junction
+		(at 207.01 69.85)
+		(diameter 0)
+		(color 0 0 0 0)
+	)
+	(junction
 		(at 203.2 135.89)
 		(diameter 0)
@@
 	)
 	(junction
-		(at 198.12 64.77)
-		(diameter 0)
-		(color 0 0 0 0)
-	)
-	(junction
 		(at 203.2 128.27)
 		(diameter 0)
@@
 	(wire
 		(pts
-			(xy 208.28 34.29) (xy 208.28 49.53)
+			(xy 208.28 34.29) (xy 208.28 45.72)
 		)
 		(stroke
@@
 	(wire
 		(pts
-			(xy 208.28 49.53) (xy 180.34 49.53)
+			(xy 208.28 45.72) (xy 180.34 45.72)
 		)
 		(stroke
@@
 	(wire
 		(pts
-			(xy 168.91 34.29) (xy 168.91 43.18)
+			(xy 168.91 34.29) (xy 168.91 38.1)
 		)
 		(stroke
@@
 	(wire
 		(pts
-			(xy 187.96 64.77) (xy 198.12 64.77)
-		)
-		(stroke
-			(width 0)
-			(type default)
-		)
-	)
-	(wire
-		(pts
 			(xy 162.56 179.07) (xy 162.56 147.32)
 		)
@@
 	(wire
 		(pts
-			(xy 198.12 64.77) (xy 207.01 64.77)
-		)
-		(stroke
-			(width 0)
-			(type default)
-		)
-	)
-	(wire
-		(pts
 			(xy 170.18 63.5) (xy 170.18 92.71)
 		)
@@
 	(wire
 		(pts
-			(xy 198.12 69.85) (xy 207.01 69.85)
-		)
-		(stroke
-			(width 0)
-			(type default)
-		)
-	)
-	(wire
-		(pts
 			(xy 111.76 113.03) (xy 111.76 105.41)
 		)
@@
 	(wire
 		(pts
-			(xy 198.12 64.77) (xy 198.12 69.85)
-		)
-		(stroke
-			(width 0)
-			(type default)
-		)
-	)
-	(wire
-		(pts
 			(xy 161.29 78.74) (xy 161.29 87.63)
 		)
@@
 	(wire
 		(pts
+			(xy 168.91 45.72) (xy 168.91 48.26)
+		)
+		(stroke
+			(width 0)
+			(type default)
+		)
+	)
+	(wire
+		(pts
 			(xy 184.15 95.25) (xy 184.15 96.52)
 		)
@@
 	(wire
 		(pts
+			(xy 186.69 64.77) (xy 207.01 64.77)
+		)
+		(stroke
+			(width 0)
+			(type default)
+		)
+	)
+	(wire
+		(pts
 			(xy 22.86 77.47) (xy 22.86 87.63)
 		)
@@
 	(wire
 		(pts
-			(xy 180.34 69.85) (xy 187.96 69.85)
+			(xy 180.34 69.85) (xy 207.01 69.85)
 		)
 		(stroke
@@
 	(wire
 		(pts
-			(xy 186.69 64.77) (xy 187.96 64.77)
-		)
-		(stroke
-			(width 0)
-			(type default)
-		)
-	)
-	(wire
-		(pts
 			(xy 111.76 105.41) (xy 119.38 105.41)
 		)
@@
 	(wire
 		(pts
-			(xy 180.34 49.53) (xy 180.34 69.85)
+			(xy 180.34 45.72) (xy 180.34 69.85)
 		)
 		(stroke
@@
 	(wire
 		(pts
-			(xy 187.96 64.77) (xy 187.96 69.85)
-		)
-		(stroke
-			(width 0)
-			(type default)
-		)
-	)
-	(wire
-		(pts
 			(xy 208.28 152.4) (xy 208.28 146.05)
 		)
@@
 	(wire
 		(pts
-			(xy 168.91 50.8) (xy 168.91 54.61)
-		)
-		(stroke
-			(width 0)
-			(type default)
-		)
-	)
-	(wire
-		(pts
 			(xy 194.31 111.76) (xy 194.31 104.14)
 		)
@@
 		)
 	)
-	(label "+3V3"
+	(label "CONN_SIG"
 		(at 213.36 69.85 180)
 		(effects
@@
 		)
 	)
-	(label "+3V3"
-		(at 208.28 34.29 0)
-		(effects
-			(font
-				(size 1.27 1.27)
-			)
-			(justify left bottom)
-		)
-	)
 	(label "I2C_SDA"
 		(at 205.74 91.44 0)
@@
 		)
 	)
-	(label "GND"
-		(at 168.91 54.61 0)
-		(effects
-			(font
-				(size 1.27 1.27)
-			)
-			(justify left bottom)
-		)
-	)
 	(label "DAC_A_CH1"
 		(at 105.41 90.17 0)
@@
 	(symbol
 		(lib_id "Device:R")
-		(at 168.91 46.99 0)
+		(at 168.91 41.91 0)
 		(unit 1)
 		(body_style 1)
@@
 		(fields_autoplaced yes)
 		(property "Reference" "R1"
-			(at 171.45 45.72 0)
+			(at 171.45 40.64 0)
 			(show_name no)
 			(do_not_autoplace no)
@@
 		)
 		(property "Value" "330"
-			(at 171.45 48.26 0)
+			(at 171.45 43.18 0)
 			(show_name no)
 			(do_not_autoplace no)
@@
 		)
 		(property "Footprint" "Resistor_THT:R_Axial_DIN0207_L6.3mm_D2.5mm_P7.62mm_Horizontal"
-			(at 167.64 46.99 90)
+			(at 167.64 41.91 90)
 			(hide yes)
 			(show_name no)
@@
 		)
 		(property "Datasheet" ""
-			(at 168.91 46.99 0)
+			(at 168.91 41.91 0)
 			(hide yes)
 			(show_name no)
@@
 		)
 		(property "Description" "Resistor"
-			(at 168.91 46.99 0)
+			(at 168.91 41.91 0)
 			(hide yes)
 			(show_name no)
@@
 		)
 		(property "KiLib_Generator" "resistor/THT"
-			(at 168.91 46.99 0)
+			(at 168.91 41.91 0)
 			(hide yes)
 			(show_name no)
@@
 			)
 		)
-		(property "Value" "SW_BOARD_CONN_LED"
+		(property "Value" "SW_BRD_CONN_SIG"
 			(at 199.39 29.21 0)
 			(show_name no)
@@
 		(fields_autoplaced yes)
 		(property "Reference" "D1"
-			(at 171.45 27.94 0)
+			(at 171.5135 27.94 0)
 			(show_name no)
 			(do_not_autoplace no)
@@
 			)
 		)
-		(property "Value" "LED_BOARD_CONN"
-			(at 171.45 30.48 0)
+		(property "Value" "LED_BRD_CONN_SIG"
+			(at 171.5135 30.48 0)
 			(show_name no)
 			(do_not_autoplace no)
@@
 					(unit 1)
 				)
+			)
+		)
+	)
+	(symbol
+		(lib_id "power:GND")
+		(at 168.91 48.26 0)
+		(unit 1)
+		(body_style 1)
+		(exclude_from_sim no)
+		(in_bom yes)
+		(on_board yes)
+		(in_pos_files yes)
+		(dnp no)
+		(fields_autoplaced yes)
+		(property "Reference" "#PWR019"
+			(at 168.91 54.61 0)
+			(hide yes)
+			(show_name no)
+			(do_not_autoplace no)
+			(effects
+				(font
+					(size 1.27 1.27)
+				)
+			)
+		)
+		(property "Value" "GND"
+			(at 168.91 53.34 0)
+			(show_name no)
+			(do_not_autoplace no)
+			(effects
+				(font
+					(size 1.27 1.27)
+				)
+			)
+		)
+		(property "Footprint" ""
+			(at 168.91 48.26 0)
+			(hide yes)
+			(show_name no)
+			(do_not_autoplace no)
+			(effects
+				(font
+					(size 1.27 1.27)
+				)
+			)
+		)
+		(property "Datasheet" ""
+			(at 168.91 48.26 0)
+			(hide yes)
+			(show_name no)
+			(do_not_autoplace no)
+			(effects
+				(font
+					(size 1.27 1.27)
+				)
+			)
+		)
+		(property "Description" "Power symbol creates a global label with name \"GND\" , ground"
+			(at 168.91 48.26 0)
+			(hide yes)
+			(show_name no)
+			(do_not_autoplace no)
+			(effects
+				(font
+					(size 1.27 1.27)
+				)
+			)
+		)
+		(pin "1"
+		)
+		(instances
+			(project "rpi-wiringpi-unit-test-platform-board-2"
+				(path "/7946ceed-5e50-51f0-9396-19e4533fa9f5"
+					(reference "#PWR019")
+					(unit 1)
+				)
